File: MCU_stm32L05/MCU_stm32L05.kicad_sch (KiCad schematic)
At the start: 28 parts, among them J1 USB_B_Micro, J2 Conn_01x04, J3 Conn_01x04, J4 Conn_01x02, J5 Conn_01x02, J6 Conn_01x02, J8 Conn_01x02, SW1 SW_SPDT, U1 STM32L052K6Tx, U2 AP2210K-3.3TRG1, Y1 32.768kHz

Commit message: update
Parts:
- added C15: 10u, Capacitor_SMD:C_0603_1608Metric, symbol Device:C
- added R2: 10k, Resistor_SMD:R_1206_3216Metric, symbol Device:R
- C1, C2, C5, C6, C7, C9: footprint (none) -> Capacitor_SMD:C_0805_2012Metric
- C10, C11, C3: footprint (none) -> Capacitor_SMD:C_0603_1608Metric
- C4, C8: footprint (none) -> Capacitor_SMD:C_1206_3216Metric
- D1: footprint (none) -> LED_SMD:LED_0603_1608Metric
- FB1, R1: footprint (none) -> Resistor_SMD:R_1206_3216Metric
- J1: footprint (none) -> Connector_USB:USB_Micro-B_Molex_47346-0001
- J2, J3: footprint (none) -> Connector_PinHeader_2.54mm:PinHeader_1x04_P2.54mm_Vertical
- J4, J5, J6, J8: footprint (none) -> Connector_PinHeader_2.54mm:PinHeader_1x02_P2.54mm_Vertical
- Y1: footprint crystal:XTAL_CC5V-T1A_32.768KHZ_12.5PF_20PPM_TA_QC -> crystal:XTAL_ABS25-32.768KHZ-6-T
Connections:
- net +3.3V: now also U1.1 (VDD), U1.17 (VDD), C15.1
- net GND: now also C15.2; no longer U1.1 (VDD), U1.17 (VDD)
- net PWR_LED: now also R2.2; no longer D1.2 (A)
- new net: D1.2 (A), R2.1
Other:
- moved on the sheet: D1
