File: usb_to_uart_ft232rl/usb_to_uart_ft232rl.kicad_pcb (KiCad board)
At the start: 4 copper layers, 20 x 32.2 mm, 14 parts, among them J1 USB_B_Micro, J2 Conn_01x05, J3 Conn_01x05, U1 FT232RL

Commit message: update
Parts:
- C1, C3: footprint Capacitor_SMD:C_0402_1005Metric -> Capacitor_SMD:C_0805_2012Metric
- J1: footprint Connector_USB:USB_Micro-B_Molex_47346-0001 -> Connector_USB:USB_Micro-B_Wuerth_629105150521
- moved J1 1.40 mm to (103.4, 64.8)
- moved C1 1.01 mm to (113.8, 54.2)
- moved C3 0.56 mm to (113.8, 57.8)
Routing:
- net VBUS: track 5.84 -> 3.88 mm
- net GND: track 21.9 -> 23.3 mm
- net /USB_D-: track 12.2 -> 11.1 mm
- net /USB_D+: track 11.5 -> 10.5 mm
- net /3V3OUT: track 2.12 -> 2.78 mm

Commit message: update
Parts:
- J1: footprint Connector_USB:USB_Micro-B_Wuerth_629105150521 -> Connector_USB:USB_Micro-B_Molex_47346-0001
- moved J1 1.50 mm to (103.4, 66.3)
Routing:
- net GND: track 23.3 -> 25.3 mm
- net VBUS: track 3.88 -> 5.82 mm
- net /USB_D-: track 11.1 -> 12.3 mm
- net /USB_D+: track 10.5 -> 11.5 mm
