File: usb_to_uart_ft232rl/usb_to_uart_ft232rl.kicad_sch (KiCad schematic)
At the start: 14 parts, among them J1 USB_B_Micro, J2 Conn_01x05, J3 Conn_01x05, U1 FT232RL

Commit message: update
Parts:
- C1, C3: footprint Capacitor_SMD:C_0402_1005Metric -> Capacitor_SMD:C_0805_2012Metric
- J1: footprint Connector_USB:USB_Micro-B_Molex_47346-0001 -> Connector_USB:USB_Micro-B_Wuerth_629105150521
Changed lines of the file:
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@@
-	(text "LED Indicators"
-		(exclude_from_sim no)
-		(at 47.752 47.244 0)
-		(effects
-			(font
-				(size 1.905 1.905)
-				(thickness 0.254)
-				(bold yes)
-			)
-		)
-	)
 	(text "LED Indicators"
 		(exclude_from_sim no)
@@
 		)
 	)
-	(text "LED Indicators"
-		(exclude_from_sim no)
-		(at 47.752 49.784 0)
-		(effects
-			(font
-				(size 1.905 1.905)
-				(thickness 0.254)
-				(bold yes)
-			)
-		)
-	)
 	(text "Connections"
 		(exclude_from_sim no)
@@
 			)
 		)
-		(property "Footprint" "Connector_USB:USB_Micro-B_Molex_47346-0001"
+		(property "Footprint" "Connector_USB:USB_Micro-B_Wuerth_629105150521"
 			(at 64.77 106.68 0)
 			(effects
@@
 			)
 		)
-		(property "Footprint" "Capacitor_SMD:C_0402_1005Metric"
+		(property "Footprint" "Capacitor_SMD:C_0805_2012Metric"
 			(at 129.2352 78.74 0)
 			(effects
@@
 			)
 		)
-		(property "Footprint" "Capacitor_SMD:C_0402_1005Metric"
+		(property "Footprint" "Capacitor_SMD:C_0805_2012Metric"
 			(at 84.7852 93.98 0)
 			(effects

Commit message: update
Parts:
- J1: footprint Connector_USB:USB_Micro-B_Wuerth_629105150521 -> Connector_USB:USB_Micro-B_Molex_47346-0001
Changed lines of the file:
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@@
 			)
 		)
-		(property "Footprint" "Connector_USB:USB_Micro-B_Wuerth_629105150521"
+		(property "Footprint" "Connector_USB:USB_Micro-B_Molex_47346-0001"
 			(at 64.77 106.68 0)
 			(effects
